Commit message: Move realsense_cam into subdirectory

File: realsense_cam/urdf/d455.urdf.xacro (robot description, xacro)
@@ -10,5 +10,5 @@
   <xacro:include filename="$(find realsense_cam)/urdf/materials.urdf.xacro" />
   <xacro:include filename="$(find realsense_cam)/urdf/usb_plug.urdf.xacro" />
-  <!--<xacro:include filename="$(find realsense_cam)/urdf/d455.gazebo.xacro"/>-->
+  <xacro:include filename="$(find realsense_cam)/urdf/d455.gazebo.xacro"/>
   <xacro:macro name="sensor_d455" params="parent *origin name:=camera use_nominal_extrinsics:=false">
     <xacro:arg name="add_plug" default="false" />
@@ -96,5 +96,5 @@
       <link name="${name}_infra1_frame"/>
       <joint name="${name}_infra1_optical_joint" type="fixed">
-        <origin xyz="0 0 0" rpy="0 0 0" />
+        <origin xyz="0 0 0" rpy="${-M_PI/2} 0 ${-M_PI/2}" />
         <parent link="${name}_infra1_frame" />
         <child link="${name}_infra1_optical_frame" />
@@ -109,5 +109,5 @@
       <link name="${name}_infra2_frame"/>
       <joint name="${name}_infra2_optical_joint" type="fixed">
-        <origin xyz="0 0 0" rpy="0 0 0" />
+        <origin xyz="0 0 0" rpy="${-M_PI/2} 0 ${-M_PI/2}" />
         <parent link="${name}_infra2_frame" />
         <child link="${name}_infra2_optical_frame" />
